File: quadparts.brd (EAGLE design)
At the start: 228.6 x 228.6 mm, 69 parts, among them J1 AVR_SPI_PRG_6NS, U1 ATMEGA128RFA1, Y1 16MHz

Commit message: Life is so hard
Parts:
- removed LED_S1, LED_S2, LED_S3, LED_S4: (no value), LEDs:LEDS
- removed R11, R13, R14, R15: 150, quadparts_prebuilt:RESC2012X60_HS
- added E$1: (no value), LEDs:LED_RING
Connections:
- removed net N$5: LED_S1.P$1, R11.2
- removed net N$6: LED_S2.P$1, R13.2
- removed net N$7: LED_S3.P$1, R14.2
- removed net N$9: LED_S4.P$1, R15.2
- removed net PB6: R14.1, U1.42
- net GND: no longer LED_S1.P$2, LED_S2.P$2, LED_S3.P$2, LED_S4.P$2
- net PB4: no longer R11.1
- net PB5: no longer R13.1
- net PB7: no longer R15.1
Routing:
- net N$6: track 106.7 -> 0.00 mm
- net N$7: track 54.5 -> 0.00 mm
- net N$9: track 48.0 -> 0.00 mm
- net N$5: track 44.6 -> 0.00 mm, vias 2 -> 0
- net GND: track 233.0 -> 202.6 mm

Commit message: I did push
Parts:
- removed C13, C15, C7, C9: 1uF, quadparts_Jason:CERAMIC_CAP_0805
- removed E$1: (no value), LEDs:LED_RING
- added C1, C2, C3, C4: 0.1uF, quadparts_prebuilt:CAPC2012X140_HS
- added LR1: (no value), LEDs:LED_RING
Connections:
- net BAT_GND: now also C1.2, C2.2, C3.2, C4.2; no longer C13.2, C15.2, C7.2, C9.2
- net N$14: now also C3.1; no longer C13.1
- net N$18: now also C4.1; no longer C15.1
- net N$2: now also C2.1; no longer C7.1
- net PB5: now also C1.1; no longer C9.1
Changed lines of the file:
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@@
 <attribute name="MPN" value="GRM21A5C2E220JW01D" x="32.258" y="37.592" size="1.778" layer="27" rot="R180" display="off"/>
 </element>
-<element name="C13" library="quadparts_Jason" package="CERAMIC_CAP_0805" value="1uF" x="-1.27" y="51.054" rot="R90">
+<element name="C3" library="quadparts_prebuilt" package="CAPC2012X140_HS" value="0.1uF" x="-1.27" y="51.054" rot="R90">
 <attribute name="CREATOR" value="SWANSON" x="-1.27" y="51.054" size="1.778" layer="27" rot="R90" display="off"/>
 <attribute name="DIST" value="Digikey" x="-1.27" y="51.054" size="1.778" layer="27" rot="R90" display="off"/>
@@
 <attribute name="MPN" value="TAJD227K006RNJ" x="-0.254" y="55.626" size="1.778" layer="27" display="off"/>
 </element>
-<element name="C15" library="quadparts_Jason" package="CERAMIC_CAP_0805" value="1uF" x="-1.016" y="-50.8" rot="R90">
+<element name="C4" library="quadparts_prebuilt" package="CAPC2012X140_HS" value="0.1uF" x="-1.016" y="-50.8" rot="R90">
 <attribute name="CREATOR" value="SWANSON" x="-1.016" y="-50.8" size="1.778" layer="27" rot="R90" display="off"/>
 <attribute name="DIST" value="Digikey" x="-1.016" y="-50.8" size="1.778" layer="27" rot="R90" display="off"/>
@@
 <attribute name="MPN" value="GRM21BR71H105KA12L" x="24.384" y="-19.558" size="1.778" layer="27" rot="R180" display="off"/>
 </element>
-<element name="C7" library="quadparts_Jason" package="CERAMIC_CAP_0805" value="1uF" x="-50.292" y="-0.762">
+<element name="C2" library="quadparts_prebuilt" package="CAPC2012X140_HS" value="0.1uF" x="-50.292" y="-0.762">
 <attribute name="CREATOR" value="SWANSON" x="-50.292" y="-0.762" size="1.778" layer="27" display="off"/>
 <attribute name="DIST" value="Digikey" x="-50.292" y="-0.762" size="1.778" layer="27" display="off"/>
@@
 <attribute name="MPN" value="GQM2195C2AR75CB01D" x="32.258" y="42.672" size="1.778" layer="27" display="off"/>
 </element>
-<element name="C9" library="quadparts_Jason" package="CERAMIC_CAP_0805" value="1uF" x="49.022" y="-3.556" rot="R180">
+<element name="C1" library="quadparts_prebuilt" package="CAPC2012X140_HS" value="0.1uF" x="49.022" y="-3.556" rot="R180">
 <attribute name="CREATOR" value="SWANSON" x="49.022" y="-3.556" size="1.778" layer="27" rot="R180" display="off"/>
 <attribute name="DIST" value="Digikey" x="49.022" y="-3.556" size="1.778" layer="27" rot="R180" display="off"/>
@@
 <attribute name="PROD_ID" value="XTAL-08218" x="-23.622" y="44.196" size="1.778" layer="27" rot="R180" display="off"/>
 </element>
-<element name="E$1" library="LEDs" package="LED_RING" value="" x="-87.122" y="61.976"/>
+<element name="LR1" library="LEDs" package="LED_RING" value="" x="-149.098" y="71.882"/>
 </elements>
 <signals>
@@
 <signal name="PB5">
 <contactref element="U1" pad="41"/>
-<contactref element="C9" pad="1"/>
+<contactref element="C1" pad="1"/>
 <contactref element="U$2" pad="P$1"/>
 <contactref element="R5" pad="2"/>
@@
 <contactref element="BREAKOUT_HEADER" pad="9"/>
 <contactref element="U$11" pad="P$2"/>
-<contactref element="C9" pad="2"/>
+<contactref element="C1" pad="2"/>
 <contactref element="U$2" pad="P$3"/>
 <contactref element="R5" pad="1"/>
-<contactref element="C7" pad="2"/>
+<contactref element="C2" pad="2"/>
 <contactref element="U$5" pad="P$3"/>
 <contactref element="R6" pad="1"/>
-<contactref element="C13" pad="2"/>
+<contactref element="C3" pad="2"/>
 <contactref element="U$7" pad="P$3"/>
 <contactref element="R8" pad="1"/>
-<contactref element="C15" pad="2"/>
+<contactref element="C4" pad="2"/>
 <contactref element="U$9" pad="P$3"/>
 <contactref element="R10" pad="1"/>
@@
 <contactref element="U$5" pad="P$1"/>
 <contactref element="R6" pad="2"/>
-<contactref element="C7" pad="1"/>
+<contactref element="C2" pad="1"/>
 <contactref element="R4" pad="2"/>
 <wire x1="-48.895" y1="3.81" x2="-48.895" y2="1.905" width="0.1524" layer="1"/>
@@
 <contactref element="R8" pad="2"/>
 <contactref element="U$7" pad="P$1"/>
-<contactref element="C13" pad="1"/>
+<contactref element="C3" pad="1"/>
 <contactref element="R7" pad="2"/>
 <wire x1="3.175" y1="52.07" x2="1.27" y2="52.07" width="0.1524" layer="1"/>
@@
 <contactref element="R10" pad="2"/>
 <contactref element="U$9" pad="P$1"/>
-<contactref element="C15" pad="1"/>
+<contactref element="C4" pad="1"/>
 <contactref element="R9" pad="2"/>
 <wire x1="3.175" y1="-49.53" x2="1.27" y2="-49.53" width="0.1524" layer="1"/>

Commit message: fix everything
Parts:
- removed C1, C2, C3, C4: 0.1uF, quadparts_prebuilt:CAPC2012X140_HS
- added C13, C15, C7, C9: 0.1uF, quadparts_Jason:CERAMIC_CAP_0805
- LR1: value (none) -> LED_RING
- moved LR1 165.5 mm to (0.00, 0.00), flipped to the bottom
Connections:
- removed net N$1: R3.2, U$3.P$4
- removed net N$28: J1.2
- new net PB6: U1.42
- net BAT_GND: now also C13.2, C15.2, C25.2, C7.2, C9.2; no longer C1.2, C2.2, C3.2, C4.2
- net GND: now also LR1.GND; no longer C25.2
- net N$14: now also C13.1; no longer C3.1
- net N$18: now also C15.1; no longer C4.1
- net N$2: now also C7.1; no longer C2.1
- net PB4: now also LR1.DATA_IN
- net PB5: now also C9.1; no longer C1.1
- net SDA: now also R3.2, U$3.P$4; no longer C17.1, R2.1, R3.1, U$3.P$1, U$3.P$13, U$3.P$3, U$3.P$5, U$3.P$6, U$3.P$7, U$3.P$8
- net V3: now also C17.1, R2.1, R3.1, U$3.P$1, U$3.P$13, U$3.P$3, U$3.P$5, U$3.P$6, U$3.P$7, U$3.P$8
- net VBAT: now also LR1.PWR
Routing:
- net GND: track 202.6 -> 201.7 mm

Commit message: minor fix the board
Parts:
- BREAKOUT_HEADER: value (none) -> NOVALUE
- moved U$1 5.55 mm to (39.4, -2.54)
- moved R5 4.19 mm to (48.0, -5.33)
- moved R12 3.94 mm to (48.0, -3.05)
- moved C9 3.59 mm to (48.5, 0.00)
- moved C19 2.96 mm to (-6.35, 5.84)
- moved R3 2.51 mm to (-6.35, -2.29)
- moved C22 2.27 mm to (4.32, 3.30)
- moved R2 2.17 mm to (-6.60, 0.76)
- moved C21 1.98 mm to (1.52, 5.84)
- moved A1 1.80 mm to (39.9, 38.9)
- moved U$8 1.55 mm to (1.52, -45.0)
- moved C17 1.55 mm to (0.25, -4.32), turned to 0 degrees
- moved C20 1.30 mm to (-2.03, 5.59)
- moved U$2 1.14 mm to (41.4, 3.56)
- moved D4 0.92 mm to (47.5, 3.81)
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Connections:
- removed net A0: U1.63
- removed net A1: U1.64
- removed net A2: U1.1
- removed net A3: U1.2
- removed net A4: U1.3
- removed net A5: U1.4
- removed net A6: U1.5
- removed net A7: U1.6
- removed net AREF: U1.62
- removed net PB6: U1.42
- removed net PB7: U1.43
- removed net PD4: U1.29
- removed net PD5: U1.30
- removed net PD6: U1.31
- removed net PD7: U1.32
- removed net PE2: U1.48
- removed net PE6: U1.52
- removed net PE7: U1.53
- removed net PG0: U1.14
- removed net PG1: U1.15
- removed net PG2: U1.16
- removed net PG5: U1.19
- removed net RSTON: U1.13
- removed net SSN: U1.36
- new net N$1: C9.1, R12.2, R5.2, U$2.P$1
- net PB5: no longer C9.1, R12.2, R5.2, U$2.P$1
Routing:
- net TX1: track 0.00 -> 102.3 mm, vias 0 -> 1
- net RX1: track 0.00 -> 99.6 mm, vias 0 -> 1
- net SDA: track 0.00 -> 89.3 mm, vias 0 -> 3
- net TX0: track 0.00 -> 85.3 mm, vias 0 -> 2
- net PE4: track 50.1 -> 126.9 mm, vias 1 -> 3
- net GND: track 201.7 -> 269.3 mm
- net V3: track 34.8 -> 97.3 mm, vias 3 -> 7
- net N$1: track 0.00 -> 28.6 mm, vias 0 -> 2
- net BAT_GND: track 319.6 -> 346.8 mm
- net PE3: track 129.1 -> 155.6 mm, vias 1 -> 3
- net MOSI: track 0.00 -> 19.9 mm, vias 0 -> 1
- net SCL: track 70.1 -> 89.4 mm, vias 0 -> 2
- net MISO: track 0.00 -> 17.3 mm, vias 0 -> 1
- net PB4: track 0.00 -> 16.7 mm, vias 0 -> 2
- net VBAT: track 298.2 -> 313.5 mm
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