File: quadcopter.sch (EAGLE design)
At the start: 62 parts, among them J1 AVR_SPI_PRG_6NS, U1 ATMEGA128RFA1, Y1 16MHz

Commit message: Renamed schematics
Connections:
- net GND: now also JP2.6

Commit message: Curently updating
Parts:
- C11, C14, C16, C18: value 100uF -> 220uF
