File: quadcopter.brd (EAGLE design)
At the start: 136.9 x 137 mm, 62 parts, among them J1 AVR_SPI_PRG_6NS, U1 ATMEGA128RFA1, Y1 16MHz

Commit message: Tapeout
Parts:
- BREAKOUT_HEADER: value NOVALUE -> N?A
- C10: value 1uF -> 0.1uF
- moved R3 1.33 mm to (-5.99, -3.67)
Connections:
- removed net N$26: C16.1, D3.C, U$8.V+
- net BAT_GND: now also C11.2, C14.2, C16.2, C18.2
- net GND: no longer C11.2, C14.2, C16.2, C18.2
- net VBAT: now also C16.1, D3.C, U$8.V+
Routing:
- net VBAT: track 116.7 -> 171.0 mm, vias 4 -> 5
- net BAT_GND: track 278.6 -> 313.2 mm
- net GND: track 246.1 -> 220.9 mm, vias 10 -> 7
- net N$26: track 12.8 -> 0.00 mm
- net V3: track 238.8 -> 248.8 mm
- net RESET: track 131.0 -> 139.2 mm
- net PE4: track 107.7 -> 104.9 mm
- net SDA: track 95.5 -> 95.8 mm, vias 2 -> 3

Commit message: Changes from first board review
Parts:
- removed D1, D2, D3, D4: 360mV, quadparts_prebuilt:SOD3716X135_HS
- added D5, D6, D7, D8: (no value), quadparts_prebuilt:SOD3716X135_HS
- moved C8 7.01 mm to (45.0, 8.97), turned to 90 degrees
- moved C21 3.41 mm to (2.34, 5.04), turned to 90 degrees
- moved C20 2.69 mm to (-2.46, 5.06)
- moved C19 2.64 mm to (-0.09, 5.08)
- moved C17 2.59 mm to (-4.96, 5.09)
- moved R3 2.29 mm to (-4.16, -2.29), turned to 90 degrees
- moved R2 1.86 mm to (-4.17, 1.21)
- moved C22 1.70 mm to (4.55, 1.75)
- moved C12 1.09 mm to (43.0, 8.96), turned to 90 degrees
- moved C5 0.60 mm to (13.6, 4.01)
- moved A1 0.51 mm to (49.9, 5.45)
- moved C24 0.13 mm to (-20.4, -0.97)
- moved C23 0.08 mm to (-20.1, 3.10)
Connections:
- net N$13: now also D6.A; no longer D1.A
- net N$16: now also D5.A; no longer D4.A
- net N$17: now also D7.A; no longer D2.A
- net N$19: now also D8.A; no longer D3.A
- net VBAT: now also D5.C, D6.C, D7.C, D8.C; no longer D1.C, D2.C, D3.C, D4.C
Routing:
- net BAT_GND: track 313.2 -> 0.00 mm, vias 2 -> 0
- net V3: track 248.8 -> 0.00 mm, vias 4 -> 0
- net GND: track 220.9 -> 0.00 mm, vias 7 -> 0
- net VBAT: track 171.0 -> 0.00 mm, vias 5 -> 0
- net PE3: track 139.9 -> 0.00 mm, vias 4 -> 0
- net RESET: track 139.2 -> 0.00 mm, vias 2 -> 0
- net PB5: track 129.5 -> 0.00 mm, vias 2 -> 0
- net PE5: track 125.8 -> 0.00 mm, vias 3 -> 0
- net PE4: track 104.9 -> 0.00 mm, vias 6 -> 0
- net SDA: track 95.8 -> 0.00 mm, vias 3 -> 0
- net SCL: track 88.9 -> 0.00 mm, vias 2 -> 0
- net TX0: track 76.5 -> 0.00 mm, vias 1 -> 0
- net TX1: track 74.1 -> 0.00 mm, vias 1 -> 0
- net RX0: track 71.3 -> 0.00 mm, vias 1 -> 0
- net RX1: track 68.9 -> 0.00 mm, vias 1 -> 0
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- added copper zone on layer 15, net BAT_GND
- added copper zone on layer 15, net N$5

Commit message: Update
Parts:
- added SW1: PUSHBUTTON_SMD-VERTICAL-1, quadparts_prebuilt:TE_FSM8JSMA_HS
- moved C26 5.34 mm to (27.3, 19.9)
- moved C27 4.26 mm to (23.8, 19.9)
- moved C29 3.28 mm to (21.0, 16.0), turned to 90 degrees
- moved Y1 2.80 mm to (25.4, 16.6), turned to 180 degrees
- moved R4 2.33 mm to (32.6, 28.4)
- moved C22 1.35 mm to (4.72, 3.09), turned to 180 degrees
- moved C7 1.32 mm to (27.9, 34.8)
- moved R6 1.07 mm to (25.4, 37.6)
- moved R3 0.89 mm to (-3.82, -1.47)
- moved C17 0.89 mm to (-4.16, 5.47)
- moved R2 0.79 mm to (-4.13, 2.00), turned to 270 degrees
- moved D6 0.66 mm to (36.7, 28.1)
- moved C21 0.59 mm to (1.92, 4.62), turned to 270 degrees
- moved C20 0.53 mm to (-2.15, 4.63)
- moved U$11 0.53 mm to (-19.0, 1.51)
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Connections:
- net RESET: now also SW1.1, SW1.2
Routing:
- net GND: track 0.00 -> 193.8 mm, vias 0 -> 17
- net V3: track 0.00 -> 186.5 mm, vias 0 -> 2
- net PE3: track 0.00 -> 135.8 mm, vias 0 -> 2
- net RESET: track 0.00 -> 117.0 mm, vias 0 -> 1
- net PB5: track 0.00 -> 116.9 mm
- net PE4: track 0.00 -> 111.7 mm, vias 0 -> 1
- net PE5: track 0.00 -> 107.4 mm, vias 0 -> 2
- net RX0: track 0.00 -> 98.2 mm
- net BAT_GND: track 0.00 -> 96.7 mm, vias 0 -> 6
- net VBAT: track 0.00 -> 96.5 mm, vias 0 -> 6
- net SDA: track 0.00 -> 89.1 mm, vias 0 -> 2
- net SCL: track 0.00 -> 86.2 mm, vias 0 -> 2
- net TX0: track 0.00 -> 77.2 mm, vias 0 -> 2
- net TX1: track 0.00 -> 70.3 mm, vias 0 -> 1
- net RX1: track 0.00 -> 68.5 mm, vias 0 -> 1
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
Commit message: Done?
Parts:
- D5, D6, D7, D8: value (none) -> 360mV
- moved J1 40.3 mm to (41.8, 22.8)
- moved R1 26.5 mm to (32.0, 14.2), turned to 180 degrees
- moved C26 25.7 mm to (23.0, -5.44)
- moved C27 25.6 mm to (27.5, -5.48)
- moved C29 19.9 mm to (30.3, -1.58), turned to 270 degrees
- moved C28 19.9 mm to (28.4, 14.2), turned to 0 degrees
- moved Y1 18.7 mm to (25.9, -2.12), turned to 0 degrees
- moved C6 13.4 mm to (20.7, -0.86)
- moved C5 4.60 mm to (18.2, 4.35), turned to 90 degrees
- moved R2 3.35 mm to (-7.47, 2.29)
- moved C22 2.93 mm to (2.09, 4.38), turned to 270 degrees
- moved C21 2.20 mm to (4.10, 4.36)
- moved R3 1.82 mm to (-5.57, -1.98)
- moved C17 1.16 mm to (-3.88, 4.34)
- moved C25 0.96 mm to (-19.0, 11.7)
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Connections:
- net BAT_GND: now also BATT1.-, U$11.P$1; no longer U$11.P$2
- net GND: now also SW1.3, SW1.4, U$11.P$2; no longer BATT1.-, U$11.P$1
Routing:
- net RX0: track 98.2 -> 61.1 mm
- net RX1: track 68.5 -> 94.6 mm, vias 1 -> 2
- net PB5: track 116.9 -> 94.7 mm
- net PB4: track 55.9 -> 35.2 mm
- net PE4: track 111.7 -> 91.6 mm, vias 1 -> 2
- net V3: track 186.5 -> 167.7 mm, vias 2 -> 0
- net TX1: track 70.3 -> 88.1 mm, vias 1 -> 2
- net PE3: track 135.8 -> 118.9 mm, vias 2 -> 1
- net N$36: track 29.4 -> 13.6 mm, vias 2 -> 0
- net N$37: track 26.1 -> 13.1 mm, vias 2 -> 0
- net VBAT: track 96.5 -> 84.3 mm, vias 6 -> 5
- net TX0: track 77.2 -> 65.2 mm, vias 2 -> 1
- net MISO: track 25.1 -> 33.5 mm
- net MOSI: track 28.1 -> 36.5 mm
- net GND: track 193.8 -> 185.8 mm
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